File: BackplaneBoard.sch (EAGLE design)
At the start: 15 parts

Commit message: V2 of Backplane
Connections:
- removed net PROG_SEL: U$2G$1.P$5, U$3G$1.P$5, U$4G$1.P$5
Changed lines of the file:
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@@
-</segment>
-</net>
-<net name="PROG_SEL" class="0">
-<segment>
-<pinref part="U$2" gate="G$1" pin="P$5"/>
-<wire x1="279.4" y1="132.08" x2="276.86" y2="132.08" width="0.1524" layer="91"/>
-<label x="271.78" y="132.08" size="1.778" layer="95"/>
-</segment>
-<segment>
-<pinref part="U$3" gate="G$1" pin="P$5"/>
-<wire x1="406.4" y1="132.08" x2="403.86" y2="132.08" width="0.1524" layer="91"/>
-<label x="398.78" y="132.08" size="1.778" layer="95"/>
-</segment>
-<segment>
-<pinref part="U$4" gate="G$1" pin="P$5"/>
-<wire x1="279.4" y1="53.34" x2="276.86" y2="53.34" width="0.1524" layer="91"/>
-<label x="271.78" y="53.34" size="1.778" layer="95"/>
 </segment>
 </net>

Commit message: Version 4
Parts:
- added U$12, U$13: T2I, BackplaneParts:T2I
Connections:
- net +5V: now also U$12.1, U$12.2, U$12.3, U$12.4
- net GND: now also U$13.1, U$13.2, U$13.3, U$13.4
Other:
- note added: "+5V Fan"
- note added: "GND Fan"

Commit message: Backplane V3
Parts:
- removed U$10, U$11, U$12, U$13, U$5, U$6, U$7, U$8, U$9: T2I, BackplaneParts:T2I
- added U$14, U$15, U$16, U$17, U$18, U$19, U$20, U$21, U$22: PHCONNECTOR, PHConnector:PHCONNECTOR
Connections:
- net +12V: now also U$17.P$1, U$17.P$2, U$17.P$3, U$17.P$4, U$20.P$1, U$20.P$2, U$20.P$3, U$20.P$4; no longer U$6.1, U$6.2, U$6.3, U$6.4, U$9.1, U$9.2, U$9.3, U$9.4
- net +5V: now also U$14.P$1, U$14.P$2, U$14.P$3, U$14.P$4, U$21.P$1, U$21.P$2, U$21.P$3, U$21.P$4; no longer U$12.1, U$12.2, U$12.3, U$12.4, U$8.1, U$8.2, U$8.3, U$8.4
- net CAN_H: now also U$16.P$2, U$19.P$2; no longer U$5.2, U$7.2
- net CAN_L: now also U$16.P$3, U$19.P$3; no longer U$5.3, U$7.3
- net GND: now also U$15.P$1, U$15.P$2, U$15.P$3, U$15.P$4, U$18.P$1, U$18.P$2, U$18.P$3, U$18.P$4, U$22.P$1, U$22.P$2, U$22.P$3, U$22.P$4; no longer U$10.1, U$10.2, U$10.3, U$10.4, U$11.1, U$11.2, U$11.3, U$11.4, U$13.1, U$13.2, U$13.3, U$13.4

Commit message: added connector
Parts:
- added U$5: PHCONNECTOR, PHConnector:PHCONNECTOR
Connections:
- new net PROG_1: U$2G$1.P$5, U$5.P$2
- new net PROG_2: U$3G$1.P$5, U$5.P$3
- new net PROG_3: U$4G$1.P$5, U$5.P$4
Other:
- note added: "Programmer"
Changed lines of the file:
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@@
 <?xml version="1.0" encoding="utf-8"?>
 <!DOCTYPE eagle SYSTEM "eagle.dtd">
-<eagle version="9.1.3">
+<eagle version="8.6.1">
 <drawing>
 <settings>
@@
 <part name="P+24" library="supply1" library_urn="urn:adsk.eagle:library:371" deviceset="+5V" device=""/>
 <part name="P+25" library="supply1" library_urn="urn:adsk.eagle:library:371" deviceset="+12V" device=""/>
+<part name="U$5" library="PHConnector" deviceset="PHCONNECTOR" device=""/>
 </parts>
 <sheets>
@@
 <text x="165.1" y="86.36" size="1.778" layer="91">+5V Fan</text>
 <text x="165.1" y="55.88" size="1.778" layer="91">GND Fan</text>
+<text x="27.94" y="104.14" size="1.778" layer="91">Programmer</text>
 </plain>
 <instances>
@@
 <instance part="P+24" gate="1" x="157.48" y="83.82"/>
 <instance part="P+25" gate="1" x="78.74" y="55.88"/>
+<instance part="U$5" gate="G$1" x="33.02" y="101.6"/>
 </instances>
 <busses>
@@
 </segment>
 </net>
+<net name="PROG_1" class="0">
+<segment>
+<pinref part="U$2" gate="G$1" pin="P$5"/>
+<wire x1="279.4" y1="132.08" x2="271.78" y2="132.08" width="0.1524" layer="91"/>
+<label x="271.78" y="132.08" size="1.778" layer="95"/>
+</segment>
+<segment>
+<pinref part="U$5" gate="G$1" pin="P$2"/>
+<wire x1="27.94" y1="93.98" x2="10.16" y2="93.98" width="0.1524" layer="91"/>
+<label x="10.16" y="93.98" size="1.778" layer="95"/>
+</segment>
+</net>
+<net name="PROG_3" class="0">
+<segment>
+<pinref part="U$4" gate="G$1" pin="P$5"/>
+<wire x1="279.4" y1="53.34" x2="274.32" y2="53.34" width="0.1524" layer="91"/>
+<label x="271.78" y="53.34" size="1.778" layer="95"/>
+</segment>
+<segment>
+<pinref part="U$5" gate="G$1" pin="P$4"/>
+<wire x1="27.94" y1="83.82" x2="10.16" y2="83.82" width="0.1524" layer="91"/>
+<label x="10.16" y="83.82" size="1.778" layer="95"/>
+</segment>
+</net>
+<net name="PROG_2" class="0">
+<segment>
+<pinref part="U$3" gate="G$1" pin="P$5"/>
+<wire x1="406.4" y1="132.08" x2="398.78" y2="132.08" width="0.1524" layer="91"/>
+<label x="396.24" y="132.08" size="1.778" layer="95"/>
+</segment>
+<segment>
+<pinref part="U$5" gate="G$1" pin="P$3"/>
+<wire x1="27.94" y1="88.9" x2="10.16" y2="88.9" width="0.1524" layer="91"/>
+<label x="10.16" y="88.9" size="1.778" layer="95"/>
+</segment>
+</net>
