File: BackplaneBoard.brd (EAGLE design)
At the start: 139.7 x 76.2 mm, 8 parts

Commit message: Added more connections to the pins
something something did something
Connections:
- new net +5V: U$1.13, U$1.14, U$1.15, U$1.16, U$1.22, U$1.23, U$1.24, U$1.5, U$1.6, U$1.7, U$1.8
- net +12V: now also U$1.P3-1, U$1.P3-2, U$1.P3-3, U$1.P3-4, U$1.P3-5, U$1.P3-6, U$1.P3-7, U$1.P3-8, U$1.P4-1, U$1.P4-2, U$1.P4-3, U$1.P4-4, U$1.P4-5, U$1.P4-6, U$1.P4-7, U$1.P4-8
- net +3V3: now also U$1.1, U$1.10, U$1.11, U$1.12, U$1.17, U$1.18, U$1.19, U$1.2, U$1.3, U$1.4, U$1.9
- net CAN_H: now also U$1.20
- net CAN_L: now also U$1.21
- net GND: now also U$1.P1-1, U$1.P1-2, U$1.P1-3, U$1.P1-4, U$1.P1-5, U$1.P1-6, U$1.P1-7, U$1.P1-8, U$1.P2-1, U$1.P2-2, U$1.P2-3, U$1.P2-4, U$1.P2-5, U$1.P2-6, U$1.P2-7, U$1.P2-8
Changed lines of the file:
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@@
 <vertex x="111" y="58"/>
 </polygon>
-<wire x1="72.39" y1="57.15" x2="102.87" y2="57.15" width="0" layer="19" extent="1-1"/>
-<wire x1="34.29" y1="57.15" x2="64.77" y2="57.15" width="0" layer="19" extent="1-1"/>
+<contactref element="U$1" pad="P1-1"/>
+<contactref element="U$1" pad="P1-2"/>
+<contactref element="U$1" pad="P1-3"/>
+<contactref element="U$1" pad="P1-4"/>
+<contactref element="U$1" pad="P2-1"/>
+<contactref element="U$1" pad="P2-2"/>
+<contactref element="U$1" pad="P2-3"/>
+<contactref element="U$1" pad="P2-4"/>
+<contactref element="U$1" pad="P1-5"/>
+<contactref element="U$1" pad="P1-6"/>
+<contactref element="U$1" pad="P1-7"/>
+<contactref element="U$1" pad="P1-8"/>
+<contactref element="U$1" pad="P2-5"/>
+<contactref element="U$1" pad="P2-6"/>
+<contactref element="U$1" pad="P2-7"/>
+<contactref element="U$1" pad="P2-8"/>
+<wire x1="11.41" y1="24.04" x2="13.91" y2="24.04" width="0" layer="19" extent="1-1"/>
+<wire x1="8.91" y1="24.04" x2="11.41" y2="24.04" width="0" layer="19" extent="1-1"/>
+<wire x1="6.41" y1="24.04" x2="8.91" y2="24.04" width="0" layer="19" extent="1-1"/>
+<wire x1="13.91" y1="21.04" x2="13.91" y2="24.04" width="0" layer="19" extent="1-1"/>
+<wire x1="11.41" y1="21.04" x2="13.91" y2="21.04" width="0" layer="19" extent="1-1"/>
+<wire x1="13.91" y1="18.54" x2="13.91" y2="21.04" width="0" layer="19" extent="1-1"/>
+<wire x1="8.91" y1="21.04" x2="11.41" y2="21.04" width="0" layer="19" extent="1-1"/>
+<wire x1="11.41" y1="18.54" x2="11.41" y2="21.04" width="0" layer="19" extent="1-1"/>
+<wire x1="6.41" y1="21.04" x2="8.91" y2="21.04" width="0" layer="19" extent="1-1"/>
+<wire x1="8.91" y1="18.54" x2="8.91" y2="21.04" width="0" layer="19" extent="1-1"/>
+<wire x1="6.41" y1="18.54" x2="6.41" y2="21.04" width="0" layer="19" extent="1-1"/>
+<wire x1="13.91" y1="15.54" x2="13.91" y2="18.54" width="0" layer="19" extent="1-1"/>
+<wire x1="11.41" y1="15.54" x2="13.91" y2="15.54" width="0" layer="19" extent="1-1"/>
+<wire x1="8.91" y1="15.54" x2="11.41" y2="15.54" width="0" layer="19" extent="1-1"/>
+<wire x1="6.41" y1="15.54" x2="8.91" y2="15.54" width="0" layer="19" extent="1-1"/>
+<wire x1="26.67" y1="54.61" x2="13.91" y2="24.04" width="0" layer="19" extent="1-1"/>
+<wire x1="64.77" y1="57.15" x2="34.29" y2="57.15" width="0" layer="19" extent="1-1"/>
+<wire x1="102.87" y1="57.15" x2="72.39" y2="57.15" width="0" layer="19" extent="1-1"/>
 <wire x1="96.52" y1="24.13" x2="102.87" y2="54.61" width="0" layer="19" extent="1-1"/>
 <wire x1="124.46" y1="24.13" x2="96.52" y2="24.13" width="0" layer="19" extent="1-1"/>
@@
 <vertex x="58" y="58"/>
 </polygon>
+<contactref element="U$1" pad="P3-5"/>
+<contactref element="U$1" pad="P4-8"/>
+<contactref element="U$1" pad="P4-7"/>
+<contactref element="U$1" pad="P4-6"/>
+<contactref element="U$1" pad="P4-5"/>
+<contactref element="U$1" pad="P3-8"/>
+<contactref element="U$1" pad="P3-7"/>
+<contactref element="U$1" pad="P3-6"/>
+<contactref element="U$1" pad="P3-1"/>
+<contactref element="U$1" pad="P4-4"/>
+<contactref element="U$1" pad="P4-3"/>
+<contactref element="U$1" pad="P4-2"/>
+<contactref element="U$1" pad="P4-1"/>
+<contactref element="U$1" pad="P3-4"/>
+<contactref element="U$1" pad="P3-3"/>
+<contactref element="U$1" pad="P3-2"/>
+<wire x1="11.41" y1="60.3" x2="13.91" y2="60.3" width="0" layer="19" extent="1-1"/>
+<wire x1="8.91" y1="60.3" x2="11.41" y2="60.3" width="0" layer="19" extent="1-1"/>
+<wire x1="6.41" y1="60.3" x2="8.91" y2="60.3" width="0" layer="19" extent="1-1"/>
+<wire x1="13.91" y1="57.3" x2="13.91" y2="60.3" width="0" layer="19" extent="1-1"/>
+<wire x1="13.91" y1="54.8" x2="13.91" y2="57.3" width="0" layer="19" extent="1-1"/>
+<wire x1="11.41" y1="57.3" x2="13.91" y2="57.3" width="0" layer="19" extent="1-1"/>
+<wire x1="11.41" y1="54.8" x2="13.91" y2="54.8" width="0" layer="19" extent="1-1"/>
+<wire x1="8.91" y1="57.3" x2="11.41" y2="57.3" width="0" layer="19" extent="1-1"/>
+<wire x1="8.91" y1="54.8" x2="11.41" y2="54.8" width="0" layer="19" extent="1-1"/>
+<wire x1="6.41" y1="57.3" x2="8.91" y2="57.3" width="0" layer="19" extent="1-1"/>
+<wire x1="6.41" y1="54.8" x2="8.91" y2="54.8" width="0" layer="19" extent="1-1"/>
+<wire x1="13.91" y1="51.8" x2="13.91" y2="54.8" width="0" layer="19" extent="1-1"/>
+<wire x1="11.41" y1="51.8" x2="13.91" y2="51.8" width="0" layer="19" extent="1-1"/>
+<wire x1="8.91" y1="51.8" x2="11.41" y2="51.8" width="0" layer="19" extent="1-1"/>
+<wire x1="6.41" y1="51.8" x2="8.91" y2="51.8" width="0" layer="19" extent="1-1"/>
+<wire x1="25.4" y1="24.13" x2="13.91" y2="51.8" width="0" layer="19" extent="1-1"/>
+<wire x1="63.5" y1="24.13" x2="35.56" y2="24.13" width="0" layer="19" extent="1-1"/>
+<wire x1="101.6" y1="24.13" x2="73.66" y2="24.13" width="0" layer="19" extent="1-1"/>
+<wire x1="57.15" y1="54.61" x2="63.5" y2="24.13" width="0" layer="19" extent="1-1"/>
 <wire x1="85.09" y1="54.61" x2="57.15" y2="54.61" width="0" layer="19" extent="1-1"/>
 <wire x1="123.19" y1="54.61" x2="95.25" y2="54.61" width="0" layer="19" extent="1-1"/>
-<wire x1="101.6" y1="24.13" x2="95.25" y2="54.61" width="0" layer="19" extent="1-1"/>
-<wire x1="73.66" y1="24.13" x2="101.6" y2="24.13" width="0" layer="19" extent="1-1"/>
-<wire x1="35.56" y1="24.13" x2="63.5" y2="24.13" width="0" layer="19" extent="1-1"/>
 </signal>
 <signal name="+3V3">
@@
 <vertex x="82" y="25"/>
 </polygon>
+<contactref element="U$1" pad="1"/>
+<contactref element="U$1" pad="4"/>
+<contactref element="U$1" pad="3"/>
+<contactref element="U$1" pad="2"/>
+<contactref element="U$1" pad="9"/>
+<contactref element="U$1" pad="10"/>
+<contactref element="U$1" pad="11"/>
+<contactref element="U$1" pad="12"/>
+<contactref element="U$1" pad="17"/>
+<contactref element="U$1" pad="18"/>
+<contactref element="U$1" pad="19"/>
+<wire x1="7.32" y1="36.83" x2="9.86" y2="36.83" width="0" layer="19" extent="1-1"/>
+<wire x1="9.86" y1="34.29" x2="9.86" y2="36.83" width="0" layer="19" extent="1-1"/>
+<wire x1="12.4" y1="34.29" x2="9.86" y2="34.29" width="0" layer="19" extent="1-1"/>
+<wire x1="12.4" y1="31.75" x2="12.4" y2="34.29" width="0" layer="19" extent="1-1"/>
+<wire x1="7.32" y1="34.29" x2="7.32" y2="36.83" width="0" layer="19" extent="1-1"/>
+<wire x1="9.86" y1="31.75" x2="9.86" y2="34.29" width="0" layer="19" extent="1-1"/>
+<wire x1="12.4" y1="29.21" x2="12.4" y2="31.75" width="0" layer="19" extent="1-1"/>
+<wire x1="7.32" y1="31.75" x2="7.32" y2="34.29" width="0" layer="19" extent="1-1"/>
+<wire x1="9.86" y1="29.21" x2="9.86" y2="31.75" width="0" layer="19" extent="1-1"/>
+<wire x1="7.32" y1="29.21" x2="7.32" y2="31.75" width="0" layer="19" extent="1-1"/>
+<wire x1="40.64" y1="24.13" x2="12.4" y2="29.21" width="0" layer="19" extent="1-1"/>
+<wire x1="78.74" y1="24.13" x2="43.18" y2="24.13" width="0" layer="19" extent="1-1"/>
 <wire x1="116.84" y1="24.13" x2="81.28" y2="24.13" width="0" layer="19" extent="1-1"/>
-<wire x1="43.18" y1="24.13" x2="78.74" y2="24.13" width="0" layer="19" extent="1-1"/>
 </signal>
 <signal name="PROG_SEL">
@@
 <contactref element="U$3" pad="P$6"/>
 <contactref element="U$4" pad="P$6"/>
+<contactref element="U$1" pad="20"/>
 <wire x1="77.47" y1="54.61" x2="115.57" y2="54.61" width="0" layer="19" extent="1-1"/>
 <wire x1="39.37" y1="54.61" x2="77.47" y2="54.61" width="0" layer="19" extent="1-1"/>
+<wire x1="12.4" y1="36.83" x2="39.37" y2="54.61" width="0" layer="19" extent="1-1"/>
 </signal>
 <signal name="CAN_L">
@@
 <contactref element="U$3" pad="P$7"/>
 <contactref element="U$4" pad="P$7"/>
+<contactref element="U$1" pad="21"/>
 <wire x1="80.01" y1="54.61" x2="118.11" y2="54.61" width="0" layer="19" extent="1-1"/>
 <wire x1="41.91" y1="54.61" x2="80.01" y2="54.61" width="0" layer="19" extent="1-1"/>
+<wire x1="12.4" y1="39.37" x2="41.91" y2="54.61" width="0" layer="19" extent="1-1"/>
+</signal>
+<signal name="+5V">
+<contactref element="U$1" pad="13"/>
+<contactref element="U$1" pad="15"/>
+<contactref element="U$1" pad="16"/>
+<contactref element="U$1" pad="14"/>
+<contactref element="U$1" pad="22"/>
+<contactref element="U$1" pad="23"/>
+<contactref element="U$1" pad="24"/>
+<contactref element="U$1" pad="5"/>
+<contactref element="U$1" pad="8"/>
+<contactref element="U$1" pad="7"/>
+<contactref element="U$1" pad="6"/>
+<wire x1="9.86" y1="46.99" x2="12.4" y2="46.99" width="0" layer="19" extent="1-1"/>
+<wire x1="12.4" y1="44.45" x2="12.4" y2="46.99" width="0" layer="19" extent="1-1"/>
+<wire x1="9.86" y1="44.45" x2="9.86" y2="46.99" width="0" layer="19" extent="1-1"/>
+<wire x1="12.4" y1="41.91" x2="12.4" y2="44.45" width="0" layer="19" extent="1-1"/>
+<wire x1="7.32" y1="46.99" x2="9.86" y2="46.99" width="0" layer="19" extent="1-1"/>
+<wire x1="9.86" y1="41.91" x2="9.86" y2="44.45" width="0" layer="19" extent="1-1"/>
+<wire x1="7.32" y1="44.45" x2="9.86" y2="44.45" width="0" layer="19" extent="1-1"/>
+<wire x1="9.86" y1="39.37" x2="9.86" y2="41.91" width="0" layer="19" extent="1-1"/>
+<wire x1="7.32" y1="41.91" x2="9.86" y2="41.91" width="0" layer="19" extent="1-1"/>
+<wire x1="7.32" y1="39.37" x2="9.86" y2="39.37" width="0" layer="19" extent="1-1"/>
 </signal>
 </signals>

Commit message: Version1 of the backplane board
Parts:
- added U$10, U$11, U$5, U$6, U$7, U$8, U$9: T2I, BackplaneParts:T2I
Connections:
- net +12V: now also U$6.1, U$6.2, U$6.3, U$6.4, U$9.1, U$9.2, U$9.3, U$9.4
- net +5V: now also U$8.1, U$8.2, U$8.3, U$8.4
- net CAN_H: now also U$5.2, U$7.2
- net CAN_L: now also U$5.3, U$7.3
- net GND: now also U$10.1, U$10.2, U$10.3, U$10.4, U$11.1, U$11.2, U$11.3, U$11.4
Routing:
- net +12V: track 106.7 -> 292.5 mm
- net GND: track 137.3 -> 317.1 mm
- net CAN_H: track 0.00 -> 161.3 mm, vias 0 -> 1
- net CAN_L: track 0.00 -> 159.7 mm
- net +3V3: track 30.5 -> 154.3 mm
- net +5V: track 0.00 -> 97.9 mm
- net PROG_SEL: track 0.00 -> 84.6 mm, vias 0 -> 4
- added copper zone on layer 1, net +3V3
- added copper zone on layer 1, net +5V
- added copper zone on layer 16, net +5V

Commit message: Made Some adjustments
Routing:
- net GND: track 317.1 -> 179.8 mm
- net +12V: track 292.5 -> 184.4 mm
- net +3V3: track 154.3 -> 123.8 mm

Commit message: V2 of Backplane
Parts:
- moved U$7 18.9 mm to (88.0, 70.6), turned to 180 degrees
- moved U$5 18.8 mm to (69.9, 70.6), turned to 180 degrees
Connections:
- removed net PROG_SEL: U$2.P$5, U$3.P$5, U$4.P$5
Routing:
- net +12V: track 184.4 -> 0.00 mm
- net GND: track 179.8 -> 0.00 mm
- net CAN_L: track 159.7 -> 286.2 mm
- net PROG_SEL: track 84.6 -> 0.00 mm, vias 4 -> 0
- net CAN_H: track 161.3 -> 183.3 mm, vias 1 -> 0
- net +3V3: track 123.8 -> 127.7 mm
- removed copper zone on layer 16, net +3V3
- removed copper zone on layer 16, net +5V
