File: BackplaneBoard.brd (EAGLE design)
At the start: 139.7 x 76.2 mm, 17 parts

Commit message: Version 2
Parts:
- moved U$13 2.09 mm to (84.0, 4.11)
- moved U$12 1.85 mm to (63.2, 4.09)
- moved U$8 1.74 mm to (44.3, 4.20)
- turned U$1 to 90 degrees
Routing:
- net +5V: track 88.1 -> 53.8 mm
- net +3V3: track 127.7 -> 122.6 mm
- net CAN_H: track 183.6 -> 178.9 mm
- net CAN_L: track 184.2 -> 180.0 mm
Other:
- board text added: "Backplane v2 Melchor De La Garza Cynthia Zatlokowicz Jacob Bobson"
- board text removed: "Backplane v1 Melchor De La Garza Cynthia Zatlokowicz Jacob Bobson"

Commit message: New V3
Parts:
- moved U$1 4.00 mm to (6.16, 38.1)
- moved U$2 3.00 mm to (22.4, 22.9)
- moved U$4 3.00 mm to (104.6, 22.9)
Routing:
- net CAN_L: track 180.0 -> 121.0 mm
- net CAN_H: track 178.9 -> 124.8 mm
- net +3V3: track 122.6 -> 95.5 mm
- net +5V: track 53.8 -> 50.8 mm

Commit message: Backplane V3
Parts:
- removed U$10, U$11, U$12, U$13, U$5, U$6, U$7, U$8, U$9: T2I, BackplaneParts:T2I
- added U$14, U$15, U$16, U$17, U$18, U$19, U$20, U$21, U$22: PHCONNECTOR, PHConnector:PHCONNECTOR
Connections:
- net +12V: now also U$17.P$1, U$17.P$2, U$17.P$3, U$17.P$4, U$20.P$1, U$20.P$2, U$20.P$3, U$20.P$4; no longer U$6.1, U$6.2, U$6.3, U$6.4, U$9.1, U$9.2, U$9.3, U$9.4
- net +5V: now also U$14.P$1, U$14.P$2, U$14.P$3, U$14.P$4, U$21.P$1, U$21.P$2, U$21.P$3, U$21.P$4; no longer U$12.1, U$12.2, U$12.3, U$12.4, U$8.1, U$8.2, U$8.3, U$8.4
- net CAN_H: now also U$16.P$2, U$19.P$2; no longer U$5.2, U$7.2
- net CAN_L: now also U$16.P$3, U$19.P$3; no longer U$5.3, U$7.3
- net GND: now also U$15.P$1, U$15.P$2, U$15.P$3, U$15.P$4, U$18.P$1, U$18.P$2, U$18.P$3, U$18.P$4, U$22.P$1, U$22.P$2, U$22.P$3, U$22.P$4; no longer U$10.1, U$10.2, U$10.3, U$10.4, U$11.1, U$11.2, U$11.3, U$11.4, U$13.1, U$13.2, U$13.3, U$13.4
Routing:
- net CAN_L: track 121.0 -> 177.6 mm
- net CAN_H: track 124.8 -> 176.7 mm
- net +3V3: track 95.5 -> 127.1 mm
- net +5V: track 50.8 -> 53.2 mm
Other:
- board text added: "Backplane v3 Melchor De La Garza Cynthia Zatlokowicz Jacob Bobson"
- board text removed: "Backplane v2 Melchor De La Garza Cynthia Zatlokowicz Jacob Bobson"

Commit message: added connector
Parts:
- added U$5: PHCONNECTOR, PHConnector:PHCONNECTOR
Connections:
- new net PROG_1: U$2.P$5, U$5.P$2
- new net PROG_2: U$3.P$5, U$5.P$3
- new net PROG_3: U$4.P$5, U$5.P$4
Routing:
- net PROG_1: track 0.00 -> 113.7 mm, vias 0 -> 3
- net PROG_2: track 0.00 -> 72.5 mm
- net PROG_3: track 0.00 -> 42.3 mm
- net CAN_H: track 176.7 -> 176.6 mm, vias 0 -> 1
Changed lines of the file:
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@@
 <?xml version="1.0" encoding="utf-8"?>
 <!DOCTYPE eagle SYSTEM "eagle.dtd">
-<eagle version="9.1.3">
+<eagle version="8.6.1">
 <drawing>
 <settings>
@@
 <setting verticaltext="up"/>
 </settings>
-<grid distance="0.0196850394" unitdist="mil" unit="mil" style="lines" multiple="1" display="yes" altdistance="5" altunitdist="mil" altunit="mil"/>
+<grid distance="5" unitdist="mil" unit="mil" style="lines" multiple="1" display="yes" altdistance="5" altunitdist="mil" altunit="mil"/>
 <layers>
 <layer number="1" name="Top" color="4" fill="1" visible="yes" active="yes"/>
@@
 <param name="checkStop" value="0"/>
 <param name="checkValues" value="0"/>
-<param name="checkNames" value="1"/>
-<param name="checkWireStubs" value="1"/>
-<param name="checkPolygonWidth" value="0"/>
 <param name="useDiameter" value="13"/>
 <param name="maxErrors" value="50"/>
@@
 <element name="U$21" library="PHConnector" package="PHCONNECTOR" value="PHCONNECTOR" x="76.985" y="7.695" rot="R180"/>
 <element name="U$22" library="PHConnector" package="PHCONNECTOR" value="PHCONNECTOR" x="96.5" y="8" rot="R180"/>
+<element name="U$5" library="PHConnector" package="PHCONNECTOR" value="PHCONNECTOR" x="127.447" y="70.7453"/>
 </elements>
 <signals>
@@
 <wire x1="16" y1="46.84815" x2="16" y2="59" width="0.254" layer="16"/>
 <wire x1="16" y1="59" x2="21" y2="64" width="0.254" layer="16"/>
-<wire x1="21" y1="64" x2="35" y2="64" width="0.254" layer="16"/>
-<wire x1="35.256" y1="64" x2="62" y2="64" width="0.254" layer="16"/>
-<wire x1="62" y1="64" x2="72.618" y2="64" width="0.254" layer="16"/>
-<wire x1="73.6675" y1="64" x2="73.82" y2="64" width="0.254" layer="16"/>
-<wire x1="73.82" y1="64" x2="76" y2="64" width="0.254" layer="16"/>
-<wire x1="76.1932" y1="64" x2="81" y2="64" width="0.254" layer="16"/>
+<wire x1="21" y1="64" x2="35.1465" y2="64" width="0.254" layer="16"/>
+<wire x1="35.1465" y1="64" x2="62.5" y2="64" width="0.254" layer="16"/>
+<wire x1="62.5" y1="64" x2="73.5615" y2="64" width="0.254" layer="16"/>
+<wire x1="73.5615" y1="64" x2="81.5" y2="64" width="0.254" layer="16"/>
 <wire x1="62.5" y1="71" x2="62.5" y2="64" width="0.254" layer="16"/>
-<wire x1="62.5" y1="64" x2="62" y2="64" width="0.254" layer="16"/>
 <wire x1="81.5" y1="71" x2="81.5" y2="64" width="0.254" layer="16"/>
-<wire x1="81.5" y1="64" x2="81" y2="64" width="0.254" layer="16"/>
 <wire x1="35.1465" y1="64" x2="35.1465" y2="55.8335" width="0.254" layer="16"/>
 <wire x1="35.1465" y1="55.8335" x2="36.37" y2="54.61" width="0.254" layer="16"/>
-<wire x1="117.3628" y1="62.2822" x2="117.3628" y2="55.8130625" width="0.254" layer="16"/>
-<wire x1="117.3628" y1="55.8130625" x2="118.5658625" y2="54.61" width="0.254" layer="16"/>
-<wire x1="115.645" y1="64" x2="115.8305" y2="63.8145" width="0.254" layer="16"/>
-<wire x1="115.8305" y1="63.8145" x2="117.3628" y2="62.2822" width="0.254" layer="16"/>
-<wire x1="118.5658625" y1="54.61" x2="118.57" y2="54.61" width="0.254" layer="16"/>
-<wire x1="76" y1="64" x2="76.1932" y2="64" width="0.254" layer="16"/>
-<wire x1="35.1465" y1="64" x2="35.256" y2="64" width="0.254" layer="16"/>
-<wire x1="35" y1="64" x2="35.1465" y2="64" width="0.254" layer="16"/>
-<wire x1="81.5" y1="64" x2="115.645" y2="64" width="0.254" layer="16"/>
-<wire x1="115.645" y1="64" x2="115.8305" y2="63.8145" width="0.254" layer="16"/>
 <wire x1="76.6459375" y1="55.8732" x2="74.3148" y2="55.8732" width="0.254" layer="16"/>
 <wire x1="77.47" y1="55.0491375" x2="76.6459375" y2="55.8732" width="0.254" layer="16"/>
 <wire x1="73.5615" y1="56.6265" x2="73.5615" y2="64" width="0.254" layer="16"/>
 <wire x1="74.3148" y1="55.8732" x2="73.5615" y2="56.6265" width="0.254" layer="16"/>
-<wire x1="73.5615" y1="64" x2="73.6675" y2="64" width="0.254" layer="16"/>
-<wire x1="72.618" y1="64" x2="73.5615" y2="64" width="0.254" layer="16"/>
 <wire x1="77.47" y1="54.61" x2="77.47" y2="55.0491375" width="0.254" layer="16"/>
+<via x="117.348" y="61.976" extent="1-16" drill="0.35"/>
+<wire x1="118.57" y1="54.61" x2="117.348" y2="55.832" width="0.254" layer="1"/>
+<wire x1="117.348" y1="55.832" x2="117.348" y2="61.976" width="0.254" layer="1"/>
+<wire x1="116.848" y1="64" x2="117.348" y2="63.5" width="0.254" layer="16"/>
+<wire x1="117.348" y1="63.5" x2="117.348" y2="61.976" width="0.254" layer="16"/>
+<wire x1="81.5" y1="64" x2="116.848" y2="64" width="0.254" layer="16"/>
 </signal>
 <signal name="CAN_L">
@@
 <wire x1="40.25" y1="7.75" x2="32" y2="16" width="2.54" layer="16"/>
 </signal>
+<signal name="PROG_1">
+<contactref element="U$2" pad="P$5"/>
+<wire x1="33.83" y1="54.61" x2="36.624" y2="51.816" width="0.2032" layer="16"/>
+<wire x1="36.624" y1="51.816" x2="56.896" y2="51.816" width="0.2032" layer="16"/>
+<via x="56.896" y="51.816" extent="1-16" drill="0.35"/>
+<wire x1="56.896" y1="51.816" x2="82.804" y2="51.816" width="0.2032" layer="1"/>
+<via x="82.804" y="51.816" extent="1-16" drill="0.35"/>
+<wire x1="82.804" y1="51.816" x2="97.282" y2="51.816" width="0.2032" layer="16"/>
+<contactref element="U$5" pad="P$2"/>
+<wire x1="97.282" y1="51.816" x2="99.949" y2="54.483" width="0.2032" layer="16"/>
+<wire x1="99.949" y1="54.483" x2="99.949" y2="59.69" width="0.2032" layer="16"/>
+<wire x1="99.949" y1="59.69" x2="100.33" y2="60.071" width="0.2032" layer="16"/>
+<via x="125.984" y="60.071" extent="1-16" drill="0.35"/>
+<wire x1="125.984" y1="60.071" x2="129.032" y2="60.071" width="0.2032" layer="1"/>
+<wire x1="129.032" y1="60.071" x2="129.413" y2="60.452" width="0.2032" layer="1"/>
+<wire x1="129.413" y1="60.452" x2="129.413" y2="70.7113" width="0.2032" layer="1"/>
+<wire x1="129.413" y1="70.7113" x2="129.447" y2="70.7453" width="0.2032" layer="1"/>
+<wire x1="100.33" y1="60.071" x2="125.984" y2="60.071" width="0.2032" layer="16"/>
+</signal>
+<signal name="PROG_3">
+<contactref element="U$4" pad="P$5"/>
+<wire x1="116.03" y1="54.61" x2="117.808" y2="52.832" width="0.2032" layer="16"/>
+<wire x1="117.808" y1="52.832" x2="137.668" y2="52.832" width="0.2032" layer="16"/>
+<contactref element="U$5" pad="P$4"/>
+<wire x1="137.668" y1="52.832" x2="137.922" y2="53.086" width="0.2032" layer="16"/>
+<wire x1="137.922" y1="61.722" x2="133.35" y2="66.294" width="0.2032" layer="16"/>
+<wire x1="133.35" y1="66.294" x2="133.35" y2="70.6483" width="0.2032" layer="16"/>
+<wire x1="133.35" y1="70.6483" x2="133.447" y2="70.7453" width="0.2032" layer="16"/>
+<wire x1="137.922" y1="53.086" x2="137.922" y2="61.722" width="0.2032" layer="16"/>
+</signal>
+<signal name="PROG_2">
+<contactref element="U$3" pad="P$5"/>
+<contactref element="U$5" pad="P$3"/>
+<wire x1="74.93" y1="54.61" x2="76.454" y2="53.086" width="0.2032" layer="16"/>
+<wire x1="76.454" y1="53.086" x2="97.282" y2="53.086" width="0.2032" layer="16"/>
+<wire x1="97.282" y1="53.086" x2="99.187" y2="54.991" width="0.2032" layer="16"/>
+<wire x1="99.187" y1="54.991" x2="99.187" y2="60.198" width="0.2032" layer="16"/>
+<wire x1="99.187" y1="60.198" x2="99.822" y2="60.833" width="0.2032" layer="16"/>
+<wire x1="130.048" y1="60.833" x2="131.445" y2="62.23" width="0.2032" layer="16"/>
+<wire x1="99.822" y1="60.833" x2="130.048" y2="60.833" width="0.2032" layer="16"/>
+<wire x1="131.445" y1="62.23" x2="131.445" y2="70.7433" width="0.2032" layer="16"/>
+<wire x1="131.445" y1="70.7433" x2="131.447" y2="70.7453" width="0.2032" layer="16"/>
+</signal>
 </signals>
-<mfgpreviewcolors>
-<mfgpreviewcolor name="soldermaskcolor" color="0xC8008000"/>
-<mfgpreviewcolor name="silkscreencolor" color="0xFFFEFEFE"/>
-<mfgpreviewcolor name="backgroundcolor" color="0xFF282828"/>
-<mfgpreviewcolor name="coppercolor" color="0xFFFFBF00"/>
-<mfgpreviewcolor name="substratecolor" color="0xFF786E46"/>
-</mfgpreviewcolors>
 </board>
 </drawing>
